Commit message: updated controller, limboactuation and controller

File: stanbot_example/stanbot.urdf (robot description, URDF)
Before this commit: robot stanbot, 31 links, 30 joints
Links:
- added link ground_link, mass 0.001
- added link right_foot_px, mass 1e-10
- added link right_foot_py, mass 1e-10
- link chest: geometry collision box size=0.28 0.2 0.32; visual mesh filename=../../../model/stanbot/meshes/visual/chest_ascii.obj
Joints:
- added joint base_prismatic_x_right: type prismatic, parent right_foot_py, child right_foot_px, origin xyz=0 0 0 rpy=0 0 0, axis 1 0 0, limit lower=-2.8973 upper=2.8973 effort=87 velocity=2.1750
- added joint base_prismatic_y_right: type prismatic, parent ground_link, child right_foot_py, origin xyz=0 0 0 rpy=0 0 0, axis 0 1 0, limit lower=-2.8973 upper=2.8973 effort=87 velocity=2.1750
- added joint base_revolute: type revolute, parent right_foot_px, child right_foot, origin xyz=0 0 0 rpy=0 0 0, axis 0 0 1, limit lower=-2.8973 upper=2.8973 effort=87 velocity=2.1750
