Commit message: limboactuation, redis keys update,simviz and limbo act controller

File: stanbot_example/limboactuation.urdf (robot description, URDF)
Before this commit: robot limboactuation, 5 links, 4 joints
Links:
- removed link HA-2
- removed link VA-2
- removed link stick
- link HA: geometry visual mesh filename=../../../model/limbot/HA.obj; visual mesh filename=../../../model/limbot/HA.obj
- link VA: geometry collision cylinder length=0.6 radius=0.025; visual cylinder length=0.6 radius=0.025
Joints:
- removed joint j2
- removed joint j3
- removed joint j4

Commit message: limboactuation urdf

File: stanbot_example/limboactuation.urdf (robot description, URDF)
Before this commit: robot limboactuation, 2 links, 1 joints
Links:
- added link ground_link, mass 0.001
Joints:
- added joint j2: type prismatic, parent HA, child VA, origin xyz=0 0 0.6 rpy=0 0 0, axis 0 0 1, limit lower=0.6 upper=0.9 effort=87 velocity=2.1750
- joint j1: axis 0 0 1 -> 1 0 0; child VA -> HA; origin xyz=0 0 0.6 rpy=0 0 0 -> xyz=0 0 0 rpy=0 0 0; parent HA -> ground_link

Commit message: limbo actuation that also slides

File: stanbot_example/limboactuation.urdf (robot description, URDF)
Before this commit: robot limboactuation, 3 links, 2 joints
Links:
- link VA: geometry collision cylinder length=0.6 radius=0.025; visual mesh filename=../../../model/limbot/Limbo_stick_brown.obj

Commit message: controller with potential field, partially working

File: stanbot_example/limboactuation.urdf (robot description, URDF)
Before this commit: robot limboactuation, 3 links, 2 joints
Links:
- link VA: geometry collision cylinder length=0.6 radius=0.025; visual mesh filename=../../../model/limbot/Limbo_stick_brown.obj
- link ground_link: mass 0.001 -> 100
Joints:
- joint j2: origin xyz=0 0 0.6 rpy=0 0 0 -> xyz=0 0 0.7 rpy=0 0 0
