Commit message: limbo actuation - 2 states

File: stanbot_angle_choosing/stanbot.urdf (robot description, URDF)
Before this commit: robot stanbot, 34 links, 33 joints
Links:
- removed link ground_link
- removed link right_foot_px
- removed link right_foot_py
- link chest: geometry visual mesh filename=../../../model/stanbot/meshes/visual/chest_ascii.obj
- link head: geometry visual mesh filename=../../../model/stanbot/meshes/visual/head_ascii.obj
Joints:
- removed joint base_prismatic_x_right
- removed joint base_prismatic_y_right
- removed joint base_revolute

File: stanbot_example/limboactuation.urdf (robot description, URDF)
Before this commit: robot limboactuation, 3 links, 2 joints
Links:
- link HA: mass 4 -> 100
- link VA: mass 4 -> 100

File: stanbot_example/stanbot_ashley.urdf (robot description, URDF)
Before this commit: robot stanbot, 34 links, 33 joints
Links:
- removed link right_foot_px
- removed link right_foot_py
- added link left_foot_ground_joint, mass 1e-10
- added link right_foot_rx, mass 1e-10
- added link right_foot_ry, mass 1e-10
- added link right_foot_rz, mass 1e-10
- link chest: geometry visual mesh filename=../../../model/stanbot/meshes/visual/chest_ascii.obj
- link head: geometry visual mesh filename=../../../model/stanbot/meshes/visual/head_ascii.obj
Joints:
- removed joint base_revolute
- added joint base_prismatic_y_left: type prismatic, parent ground_link, child left_foot_ground_joint, origin xyz=0 0 0 rpy=0 0 0, axis 0 1 0, limit lower=-2.8973 upper=2.8973 effort=87 velocity=2.1750
- added joint base_prismatic_z_right: type prismatic, parent right_foot, child right_foot_ry, origin xyz=0 0 0 rpy=0 0 0, axis 0 0 1, limit lower=-2.8973 upper=2.8973 effort=87 velocity=2.1750
- joint base_prismatic_x_right: child right_foot_px -> right_foot_rx; parent right_foot_py -> right_foot_rz
- joint base_prismatic_y_right: axis 0 1 0 -> 0 0 1; child right_foot_py -> right_foot_rz
